Commit message: add pd controller

File: descriptions/go2_description/xacro/ros2_control.xacro (robot description, xacro)
@@ -8,5 +8,5 @@
             <command_interface name="position"/>
             <command_interface name="velocity"/>
-            <command_interface name="effort"/>
+            <command_interface name="torque"/>
             <command_interface name="kp"/>
             <command_interface name="kd"/>
@@ -18,5 +18,5 @@
             <command_interface name="position"/>
             <command_interface name="velocity"/>
-            <command_interface name="effort"/>
+            <command_interface name="torque"/>
             <command_interface name="kp"/>
             <command_interface name="kd"/>
@@ -28,5 +28,5 @@
             <command_interface name="position"/>
             <command_interface name="velocity"/>
-            <command_interface name="effort"/>
+            <command_interface name="torque"/>
             <command_interface name="kp"/>
             <command_interface name="kd"/>
@@ -38,5 +38,5 @@
             <command_interface name="position"/>
             <command_interface name="velocity"/>
-            <command_interface name="effort"/>
+            <command_interface name="torque"/>
             <command_interface name="kp"/>
             <command_interface name="kd"/>
@@ -48,5 +48,5 @@
             <command_interface name="position"/>
             <command_interface name="velocity"/>
-            <command_interface name="effort"/>
+            <command_interface name="torque"/>
             <command_interface name="kp"/>
             <command_interface name="kd"/>
@@ -58,5 +58,5 @@
             <command_interface name="position"/>
             <command_interface name="velocity"/>
-            <command_interface name="effort"/>
+            <command_interface name="torque"/>
             <command_interface name="kp"/>
             <command_interface name="kd"/>
@@ -68,5 +68,5 @@
             <command_interface name="position"/>
             <command_interface name="velocity"/>
-            <command_interface name="effort"/>
+            <command_interface name="torque"/>
             <command_interface name="kp"/>
             <command_interface name="kd"/>
@@ -78,5 +78,5 @@
             <command_interface name="position"/>
             <command_interface name="velocity"/>
-            <command_interface name="effort"/>
+            <command_interface name="torque"/>
             <command_interface name="kp"/>
             <command_interface name="kd"/>
@@ -88,5 +88,5 @@
             <command_interface name="position"/>
             <command_interface name="velocity"/>
-            <command_interface name="effort"/>
+            <command_interface name="torque"/>
             <command_interface name="kp"/>
             <command_interface name="kd"/>
@@ -98,5 +98,5 @@
             <command_interface name="position"/>
             <command_interface name="velocity"/>
-            <command_interface name="effort"/>
+            <command_interface name="torque"/>
             <command_interface name="kp"/>
             <command_interface name="kd"/>
@@ -108,5 +108,5 @@
             <command_interface name="position"/>
             <command_interface name="velocity"/>
-            <command_interface name="effort"/>
+            <command_interface name="torque"/>
             <command_interface name="kp"/>
             <command_interface name="kd"/>
@@ -118,5 +118,5 @@
             <command_interface name="position"/>
             <command_interface name="velocity"/>
-            <command_interface name="effort"/>
+            <command_interface name="torque"/>
             <command_interface name="kp"/>
             <command_interface name="kd"/>

File: descriptions/quadruped_gazebo/urdf/common/ros2_control.xacro (robot description, xacro)
@@ -12,5 +12,29 @@
             <state_interface name="effort"/>
         </joint>
+        <joint name="RF_HFE">
+            <command_interface name="effort" initial_value="0.0"/>
+            <state_interface name="position"/>
+            <state_interface name="velocity"/>
+            <state_interface name="effort"/>
+        </joint>
+        <joint name="RF_KFE">
+            <command_interface name="effort" initial_value="0.0"/>
+            <state_interface name="position"/>
+            <state_interface name="velocity"/>
+            <state_interface name="effort"/>
+        </joint>
         <joint name="LF_HAA">
+            <command_interface name="effort" initial_value="0.0"/>
+            <state_interface name="position"/>
+            <state_interface name="velocity"/>
+            <state_interface name="effort"/>
+        </joint>
+        <joint name="LF_HFE">
+            <command_interface name="effort" initial_value="0.0"/>
+            <state_interface name="position"/>
+            <state_interface name="velocity"/>
+            <state_interface name="effort"/>
+        </joint>
+        <joint name="LF_KFE">
             <command_interface name="effort" initial_value="0.0"/>
             <state_interface name="position"/>
@@ -24,4 +48,16 @@
             <state_interface name="effort"/>
         </joint>
+        <joint name="RH_HFE">
+            <command_interface name="effort" initial_value="0.0"/>
+            <state_interface name="position"/>
+            <state_interface name="velocity"/>
+            <state_interface name="effort"/>
+        </joint>
+        <joint name="RH_KFE">
+            <command_interface name="effort" initial_value="0.0"/>
+            <state_interface name="position"/>
+            <state_interface name="velocity"/>
+            <state_interface name="effort"/>
+        </joint>
         <joint name="LH_HAA">
             <command_interface name="effort" initial_value="0.0"/>
@@ -30,41 +66,5 @@
             <state_interface name="effort"/>
         </joint>
-        <joint name="RF_HFE">
-            <command_interface name="effort" initial_value="0.0"/>
-            <state_interface name="position"/>
-            <state_interface name="velocity"/>
-            <state_interface name="effort"/>
-        </joint>
-        <joint name="LF_HFE">
-            <command_interface name="effort" initial_value="0.0"/>
-            <state_interface name="position"/>
-            <state_interface name="velocity"/>
-            <state_interface name="effort"/>
-        </joint>
-        <joint name="RH_HFE">
-            <command_interface name="effort" initial_value="0.0"/>
-            <state_interface name="position"/>
-            <state_interface name="velocity"/>
-            <state_interface name="effort"/>
-        </joint>
         <joint name="LH_HFE">
-            <command_interface name="effort" initial_value="0.0"/>
-            <state_interface name="position"/>
-            <state_interface name="velocity"/>
-            <state_interface name="effort"/>
-        </joint>
-        <joint name="RF_KFE">
-            <command_interface name="effort" initial_value="0.0"/>
-            <state_interface name="position"/>
-            <state_interface name="velocity"/>
-            <state_interface name="effort"/>
-        </joint>
-        <joint name="LF_KFE">
-            <command_interface name="effort" initial_value="0.0"/>
-            <state_interface name="position"/>
-            <state_interface name="velocity"/>
-            <state_interface name="effort"/>
-        </joint>
-        <joint name="RH_KFE">
             <command_interface name="effort" initial_value="0.0"/>
             <state_interface name="position"/>

Commit message: can visualize and control gazebo robots

File: descriptions/go2_description/xacro/ros2_control.xacro (robot description, xacro)
@@ -8,5 +8,5 @@
             <command_interface name="position"/>
             <command_interface name="velocity"/>
-            <command_interface name="torque"/>
+            <command_interface name="effort"/>
             <command_interface name="kp"/>
             <command_interface name="kd"/>
@@ -18,5 +18,5 @@
             <command_interface name="position"/>
             <command_interface name="velocity"/>
-            <command_interface name="torque"/>
+            <command_interface name="effort"/>
             <command_interface name="kp"/>
             <command_interface name="kd"/>
@@ -28,5 +28,5 @@
             <command_interface name="position"/>
             <command_interface name="velocity"/>
-            <command_interface name="torque"/>
+            <command_interface name="effort"/>
             <command_interface name="kp"/>
             <command_interface name="kd"/>
@@ -38,5 +38,5 @@
             <command_interface name="position"/>
             <command_interface name="velocity"/>
-            <command_interface name="torque"/>
+            <command_interface name="effort"/>
             <command_interface name="kp"/>
             <command_interface name="kd"/>
@@ -48,5 +48,5 @@
             <command_interface name="position"/>
             <command_interface name="velocity"/>
-            <command_interface name="torque"/>
+            <command_interface name="effort"/>
             <command_interface name="kp"/>
             <command_interface name="kd"/>
@@ -58,5 +58,5 @@
             <command_interface name="position"/>
             <command_interface name="velocity"/>
-            <command_interface name="torque"/>
+            <command_interface name="effort"/>
             <command_interface name="kp"/>
             <command_interface name="kd"/>
@@ -68,5 +68,5 @@
             <command_interface name="position"/>
             <command_interface name="velocity"/>
-            <command_interface name="torque"/>
+            <command_interface name="effort"/>
             <command_interface name="kp"/>
             <command_interface name="kd"/>
@@ -78,5 +78,5 @@
             <command_interface name="position"/>
             <command_interface name="velocity"/>
-            <command_interface name="torque"/>
+            <command_interface name="effort"/>
             <command_interface name="kp"/>
             <command_interface name="kd"/>
@@ -88,5 +88,5 @@
             <command_interface name="position"/>
             <command_interface name="velocity"/>
-            <command_interface name="torque"/>
+            <command_interface name="effort"/>
             <command_interface name="kp"/>
             <command_interface name="kd"/>
@@ -98,5 +98,5 @@
             <command_interface name="position"/>
             <command_interface name="velocity"/>
-            <command_interface name="torque"/>
+            <command_interface name="effort"/>
             <command_interface name="kp"/>
             <command_interface name="kd"/>
@@ -108,5 +108,5 @@
             <command_interface name="position"/>
             <command_interface name="velocity"/>
-            <command_interface name="torque"/>
+            <command_interface name="effort"/>
             <command_interface name="kp"/>
             <command_interface name="kd"/>
@@ -118,5 +118,5 @@
             <command_interface name="position"/>
             <command_interface name="velocity"/>
-            <command_interface name="torque"/>
+            <command_interface name="effort"/>
             <command_interface name="kp"/>
             <command_interface name="kd"/>

File: descriptions/quadruped_gazebo/urdf/common/leg.xacro (robot description, xacro)
@@ -5,5 +5,5 @@
         <joint name="${prefix}_HAA" type="revolute">
             <xacro:insert_block name="origin"/>
-            <parent link="base"/>
+            <parent link="trunk"/>
             <child link="${prefix}_hip"/>
             <axis xyz="1 0 0"/>
@@ -36,5 +36,5 @@
                           scale="1 1 1"/>
                 </geometry>
-                <material name="orange"/>
+<!--                <material name="orange"/>-->
             </visual>
             <collision>
@@ -75,5 +75,5 @@
                     </xacro:if>
                 </geometry>
-                <material name="orange"/>
+<!--                <material name="orange"/>-->
             </visual>
             <collision>
@@ -113,5 +113,5 @@
                           scale="1 1 1"/>
                 </geometry>
-                <material name="orange"/>
+<!--                <material name="orange"/>-->
             </visual>
             <collision>
@@ -141,5 +141,5 @@
                     <sphere radius="${foot_radius-0.01}"/>
                 </geometry>
-                <material name="orange"/>
+<!--                <material name="orange"/>-->
             </visual>
             <collision>
@@ -166,5 +166,9 @@
             <mu1>0.2</mu1>
             <mu2>0.2</mu2>
-            <material>Gazebo/DarkGrey</material>
+            <material>
+                <ambient>.175 .175 .175  1.0</ambient>
+                <diffuse>.175 .175 .175  1.0</diffuse>
+                <specular>.175 .175 .175 1.000000 1.500000</specular>
+            </material>
         </gazebo>
         <gazebo reference="${prefix}_thigh">
@@ -172,5 +176,9 @@
             <mu2>0.2</mu2>
             <self_collide>0</self_collide>
-            <material>Gazebo/DarkGrey</material>
+            <material>
+                <ambient>.175 .175 .175  1.0</ambient>
+                <diffuse>.175 .175 .175  1.0</diffuse>
+                <specular>.175 .175 .175 1.000000 1.500000</specular>
+            </material>
             <kp value="1000000.0"/>
             <kd value="100.0"/>
@@ -180,4 +188,9 @@
             <mu2>0.6</mu2>
             <self_collide>1</self_collide>
+            <material>
+                <ambient>.175 .175 .175  1.0</ambient>
+                <diffuse>.175 .175 .175  1.0</diffuse>
+                <specular>.175 .175 .175 1.000000 1.500000</specular>
+            </material>
         </gazebo>
         <gazebo reference="${prefix}_FOOT">
@@ -185,5 +198,9 @@
             <mu2>0.6</mu2>
             <self_collide>1</self_collide>
-            <material>Gazebo/DarkGrey</material>
+            <material>
+                <ambient>.175 .175 .175  1.0</ambient>
+                <diffuse>.175 .175 .175  1.0</diffuse>
+                <specular>.175 .175 .175 1.000000 1.500000</specular>
+            </material>
             <kp value="1000000.0"/>
             <kd value="100.0"/>

File: descriptions/quadruped_gazebo/urdf/go1/const.xacro (robot description, xacro)
@@ -109,3 +109,10 @@
     <!-- foot -->
     <xacro:property name="foot_mass" value="0.06"/>
+    <gazebo reference="trunk">
+        <material>
+            <ambient>.175 .175 .175  1.0</ambient>
+            <diffuse>.175 .175 .175  1.0</diffuse>
+            <specular>.175 .175 .175 1.000000 1.500000</specular>
+        </material>
+    </gazebo>
 </robot>

File: descriptions/quadruped_gazebo/urdf/robot.xacro (robot description, xacro)
@@ -9,4 +9,17 @@
     <xacro:property name="mesh_path" value="file://$(find quadruped_gazebo)/meshes/$(arg robot_type)"/>
     <link name="base">
+        <visual>
+            <origin rpy="0 0 0" xyz="0 0 0"/>
+            <geometry>
+                <box size="0.001 0.001 0.001"/>
+            </geometry>
+        </visual>
+    </link>
+    <joint name="floating_base" type="fixed">
+        <origin rpy="0 0 0" xyz="0 0 0"/>
+        <parent link="base"/>
+        <child link="trunk"/>
+    </joint>
+    <link name="trunk">
         <visual>
             <origin rpy="0 0 0" xyz="0 0 0"/>
@@ -30,5 +43,5 @@
         </inertial>
     </link>
-    <xacro:IMU connected_to="base" imu_name="base_imu" xyz="0. 0. 0." rpy="0. 0. 0."/>
+    <xacro:IMU connected_to="trunk" imu_name="base_imu" xyz="0. 0. 0." rpy="0. 0. 0."/>
     <xacro:leg prefix="LF" mesh_path="${mesh_path}" mirror="1" mirror_dae="True" front_hind="1" front_hind_dae="True">
         <origin rpy="0 0 0" xyz="${leg_offset_x} ${leg_offset_y} 0"/>
