Commit message: fix go1 gazebo visualization

File: descriptions/quadruped_gazebo/urdf/common/leg.xacro (robot description, xacro)
@@ -166,9 +166,11 @@
             <mu1>0.2</mu1>
             <mu2>0.2</mu2>
-            <material>
-                <ambient>.175 .175 .175  1.0</ambient>
-                <diffuse>.175 .175 .175  1.0</diffuse>
-                <specular>.175 .175 .175 1.000000 1.500000</specular>
-            </material>
+            <visual>
+                <material>
+                    <ambient>.5 .5 .5  1.0</ambient>
+                    <diffuse>.5 .5 .5  1.0</diffuse>
+                    <specular>.5 .5 .5  1.0</specular>
+                </material>
+            </visual>
         </gazebo>
         <gazebo reference="${prefix}_thigh">
@@ -176,9 +178,11 @@
             <mu2>0.2</mu2>
             <self_collide>0</self_collide>
-            <material>
-                <ambient>.175 .175 .175  1.0</ambient>
-                <diffuse>.175 .175 .175  1.0</diffuse>
-                <specular>.175 .175 .175 1.000000 1.500000</specular>
-            </material>
+            <visual>
+                <material>
+                    <ambient>.175 .175 .175  1.0</ambient>
+                    <diffuse>.175 .175 .175  1.0</diffuse>
+                    <specular>.175 .175 .175 1.0</specular>
+                </material>
+            </visual>
             <kp value="1000000.0"/>
             <kd value="100.0"/>
@@ -188,9 +192,11 @@
             <mu2>0.6</mu2>
             <self_collide>1</self_collide>
-            <material>
-                <ambient>.175 .175 .175  1.0</ambient>
-                <diffuse>.175 .175 .175  1.0</diffuse>
-                <specular>.175 .175 .175 1.000000 1.500000</specular>
-            </material>
+            <visual>
+                <material>
+                    <ambient>.5 .5 .5  1.0</ambient>
+                    <diffuse>.5 .5 .5  1.0</diffuse>
+                    <specular>.5 .5 .5  1.0</specular>
+                </material>
+            </visual>
         </gazebo>
         <gazebo reference="${prefix}_FOOT">
@@ -198,9 +204,11 @@
             <mu2>0.6</mu2>
             <self_collide>1</self_collide>
-            <material>
-                <ambient>.175 .175 .175  1.0</ambient>
-                <diffuse>.175 .175 .175  1.0</diffuse>
-                <specular>.175 .175 .175 1.000000 1.500000</specular>
-            </material>
+            <visual>
+                <material>
+                    <ambient>.175 .175 .175  1.0</ambient>
+                    <diffuse>.175 .175 .175  1.0</diffuse>
+                    <specular>.175 .175 .175 1.0</specular>
+                </material>
+            </visual>
             <kp value="1000000.0"/>
             <kd value="100.0"/>

File: descriptions/quadruped_gazebo/urdf/common/ros2_control.xacro (robot description, xacro)
@@ -118,5 +118,5 @@
     <gazebo>
         <plugin filename="gz_ros2_control-system" name="gz_ros2_control::GazeboSimROS2ControlPlugin">
-            <parameters>$(find quadruped_gazebo)/config/jtc.yaml</parameters>
+            <parameters>$(find quadruped_gazebo)/config/robot_control.yaml</parameters>
         </plugin>
         <plugin filename="gz-sim-imu-system"

File: descriptions/quadruped_gazebo/urdf/go1/const.xacro (robot description, xacro)
@@ -110,9 +110,11 @@
     <xacro:property name="foot_mass" value="0.06"/>
     <gazebo reference="trunk">
-        <material>
-            <ambient>.175 .175 .175  1.0</ambient>
-            <diffuse>.175 .175 .175  1.0</diffuse>
-            <specular>.175 .175 .175 1.000000 1.500000</specular>
-        </material>
+        <visual name="DarkGrey">
+            <material>
+                <ambient>.5 .5 .5  1.0</ambient>
+                <diffuse>.5 .5 .5  1.0</diffuse>
+                <specular>.5 .5 .5  1.0</specular>
+            </material>
+        </visual>
     </gazebo>
 </robot>
