Commit message: add visualizer

File: descriptions/aliengo_description/urdf/robot.urdf (robot description, URDF)
Before this commit: robot aliengo, 31 links, 30 joints
Joints:
- joint FL_thigh_joint: limit effort=35.278 velocity=20 -> lower=-2.0943951023931953 upper=4.1887902047863905 effort=35.278 velocity=20
- joint FR_thigh_joint: limit effort=35.278 velocity=20 -> lower=-2.0943951023931953 upper=4.1887902047863905 effort=35.278 velocity=20
- joint RL_thigh_joint: limit effort=35.278 velocity=20 -> lower=-2.0943951023931953 upper=4.1887902047863905 effort=35.278 velocity=20
- joint RR_thigh_joint: limit effort=35.278 velocity=20 -> lower=-2.0943951023931953 upper=4.1887902047863905 effort=35.278 velocity=20

File: descriptions/aliengo_description/xacro/leg.xacro (robot description, xacro)
@@ -102,5 +102,6 @@
       <axis xyz="0 1 0"/>
       <dynamics damping="${damping}" friction="${friction}"/>
-      <limit effort="${thigh_torque_max}" velocity="${thigh_velocity_max}"/>
+      <limit effort="${thigh_torque_max}" velocity="${thigh_velocity_max}" lower="${thigh_position_min}"
+             upper="${thigh_position_max}"/>
     </joint>
     <joint name="${name}_thigh_rotor_joint" type="fixed">
