Commit message: rl controller enhanced

File: descriptions/unitree/a1_description/xacro/const.xacro (robot description, xacro)
@@ -29,6 +29,6 @@
     <xacro:property name="hip_offset" value="0.065"/>
     <!-- joint limits -->
-    <xacro:property name="damping" value="0"/>
-    <xacro:property name="friction" value="0"/>
+    <xacro:property name="damping" value="0.1"/>
+    <xacro:property name="friction" value="0.1"/>
     <xacro:property name="hip_max" value="46"/>
     <xacro:property name="hip_min" value="-46"/>

File: descriptions/unitree/a1_description/xacro/gazebo_classic.xacro (robot description, xacro)
@@ -92,5 +92,5 @@
   <gazebo>
     <plugin filename="libgazebo_ros2_control.so" name="gazebo_ros2_control">
-      <parameters>$(find go2_description)/config/gazebo.yaml</parameters>
+      <parameters>$(find a1_description)/config/gazebo.yaml</parameters>
     </plugin>
   </gazebo>

File: descriptions/unitree/a1_description/xacro/robot.xacro (robot description, xacro)
@@ -10,8 +10,8 @@
     <xacro:if value="$(arg GAZEBO)">
         <xacro:if value="$(arg CLASSIC)">
-            <xacro:include filename="$(find go2_description)/xacro/gazebo_classic.xacro"/>
+            <xacro:include filename="$(find a1_description)/xacro/gazebo_classic.xacro"/>
         </xacro:if>
          <xacro:unless value="$(arg CLASSIC)">
-              <xacro:include filename="$(find go2_description)/xacro/gazebo.xacro"/>
+              <xacro:include filename="$(find a1_description)/xacro/gazebo.xacro"/>
           </xacro:unless>
     </xacro:if>
