Commit message: tried go2 rl control but failed

File: descriptions/unitree/a1_description/xacro/gazebo.xacro (robot description, xacro)
@@ -102,11 +102,4 @@
     <mu2>0.6</mu2>
     <self_collide>1</self_collide>
-    <visual>
-      <material>
-        <ambient>.05 .05 .05 1.0</ambient>
-        <diffuse>.05 .05 .05 1.0</diffuse>
-        <specular>.05 .05 .05 1.0</specular>
-      </material>
-    </visual>
   </gazebo>
   <gazebo reference="imu_link">
@@ -119,52 +112,52 @@
         <angular_velocity>
           <x>
-<!--            <noise type="gaussian">-->
-<!--              <mean>0.0</mean>-->
-<!--              <stddev>2e-4</stddev>-->
-<!--              <bias_mean>0.0000075</bias_mean>-->
-<!--              <bias_stddev>0.0000008</bias_stddev>-->
-<!--            </noise>-->
+            <noise type="gaussian">
+              <mean>0.0</mean>
+              <stddev>2e-4</stddev>
+              <bias_mean>0.0000075</bias_mean>
+              <bias_stddev>0.0000008</bias_stddev>
+            </noise>
           </x>
           <y>
-<!--            <noise type="gaussian">-->
-<!--              <mean>0.0</mean>-->
-<!--              <stddev>2e-4</stddev>-->
-<!--              <bias_mean>0.0000075</bias_mean>-->
-<!--              <bias_stddev>0.0000008</bias_stddev>-->
-<!--            </noise>-->
+            <noise type="gaussian">
+              <mean>0.0</mean>
+              <stddev>2e-4</stddev>
+              <bias_mean>0.0000075</bias_mean>
+              <bias_stddev>0.0000008</bias_stddev>
+            </noise>
           </y>
           <z>
-<!--            <noise type="gaussian">-->
-<!--              <mean>0.0</mean>-->
-<!--              <stddev>2e-4</stddev>-->
-<!--              <bias_mean>0.0000075</bias_mean>-->
-<!--              <bias_stddev>0.0000008</bias_stddev>-->
-<!--            </noise>-->
+            <noise type="gaussian">
+              <mean>0.0</mean>
+              <stddev>2e-4</stddev>
+              <bias_mean>0.0000075</bias_mean>
+              <bias_stddev>0.0000008</bias_stddev>
+            </noise>
           </z>
         </angular_velocity>
         <linear_acceleration>
           <x>
-<!--            <noise type="gaussian">-->
-<!--              <mean>0.0</mean>-->
-<!--              <stddev>1.7e-2</stddev>-->
-<!--              <bias_mean>0.1</bias_mean>-->
-<!--              <bias_stddev>0.001</bias_stddev>-->
-<!--            </noise>-->
+            <noise type="gaussian">
+              <mean>0.0</mean>
+              <stddev>1.7e-2</stddev>
+              <bias_mean>0.1</bias_mean>
+              <bias_stddev>0.001</bias_stddev>
+            </noise>
           </x>
           <y>
-<!--            <noise type="gaussian">-->
-<!--              <mean>0.0</mean>-->
-<!--              <stddev>1.7e-2</stddev>-->
-<!--              <bias_mean>0.1</bias_mean>-->
-<!--              <bias_stddev>0.001</bias_stddev>-->
-<!--            </noise>-->
+            <noise type="gaussian">
+              <mean>0.0</mean>
+              <stddev>1.7e-2</stddev>
+              <bias_mean>0.1</bias_mean>
+              <bias_stddev>0.001</bias_stddev>
+            </noise>
           </y>
           <z>
-<!--            <noise type="gaussian">-->
-<!--              <mean>0.0</mean>-->
-<!--              <stddev>1.7e-2</stddev>-->
-<!--              <bias_mean>0.1</bias_mean>-->
-<!--              <bias_stddev>0.001</bias_stddev>-->
-<!--            </noise>-->
+            <noise type="gaussian">
+              <mean>0.0</mean>
+              <stddev>1.7e-2</stddev>
+              <bias_mean>0.1</bias_mean>
+              <bias_stddev>0.001</bias_stddev>
+            </noise>
           </z>
         </linear_acceleration>

File: descriptions/unitree/a1_description/xacro/leg.xacro (robot description, xacro)
@@ -161,11 +161,4 @@
 			<mu1>0.2</mu1>
 			<mu2>0.2</mu2>
-			<visual>
-				<material>
-					<ambient>.5 .5 .5 1.0</ambient>
-					<diffuse>.5 .5 .5 1.0</diffuse>
-					<specular>.5 .5 .5 1.0</specular>
-				</material>
-			</visual>
 		</gazebo>
 		<gazebo reference="${name}_thigh">
@@ -173,11 +166,4 @@
 			<mu2>0.2</mu2>
 			<self_collide>0</self_collide>
-			<visual>
-				<material>
-					<ambient>.175 .175 .175 1.0</ambient>
-					<diffuse>.175 .175 .175 1.0</diffuse>
-					<specular>.175 .175 .175 1.0</specular>
-				</material>
-			</visual>
 			<kp value="1000000.0"/>
 			<kd value="100.0"/>
@@ -187,11 +173,4 @@
 			<mu2>0.6</mu2>
 			<self_collide>1</self_collide>
-			<visual>
-				<material>
-					<ambient>.5 .5 .5 1.0</ambient>
-					<diffuse>.5 .5 .5 1.0</diffuse>
-					<specular>.5 .5 .5 1.0</specular>
-				</material>
-			</visual>
 		</gazebo>
 		<gazebo reference="${name}_foot">
@@ -199,11 +178,4 @@
 			<mu2>0.6</mu2>
 			<self_collide>1</self_collide>
-			<visual>
-				<material>
-					<ambient>.175 .175 .175 1.0</ambient>
-					<diffuse>.175 .175 .175 1.0</diffuse>
-					<specular>.175 .175 .175 1.0</specular>
-				</material>
-			</visual>
 			<kp value="1000000.0"/>
 			<kd value="100.0"/>

File: descriptions/unitree/a1_description/xacro/robot.xacro (robot description, xacro)
@@ -44,5 +44,4 @@
                 <mesh filename="file://$(find a1_description)/meshes/trunk.dae" scale="1 1 1"/>
             </geometry>
-            <material name="orange"/>
         </visual>
         <collision>

File: descriptions/unitree/go2_description/xacro/gazebo.xacro (robot description, xacro)
@@ -92,5 +92,5 @@
   <gazebo>
     <plugin filename="gz_ros2_control-system" name="gz_ros2_control::GazeboSimROS2ControlPlugin">
-      <parameters>$(find a1_description)/config/gazebo.yaml</parameters>
+      <parameters>$(find go2_description)/config/gazebo.yaml</parameters>
     </plugin>
     <plugin filename="gz-sim-imu-system"
@@ -112,52 +112,52 @@
         <angular_velocity>
           <x>
-<!--            <noise type="gaussian">-->
-<!--              <mean>0.0</mean>-->
-<!--              <stddev>2e-4</stddev>-->
-<!--              <bias_mean>0.0000075</bias_mean>-->
-<!--              <bias_stddev>0.0000008</bias_stddev>-->
-<!--            </noise>-->
+            <noise type="gaussian">
+              <mean>0.0</mean>
+              <stddev>2e-4</stddev>
+              <bias_mean>0.0000075</bias_mean>
+              <bias_stddev>0.0000008</bias_stddev>
+            </noise>
           </x>
           <y>
-<!--            <noise type="gaussian">-->
-<!--              <mean>0.0</mean>-->
-<!--              <stddev>2e-4</stddev>-->
-<!--              <bias_mean>0.0000075</bias_mean>-->
-<!--              <bias_stddev>0.0000008</bias_stddev>-->
-<!--            </noise>-->
+            <noise type="gaussian">
+              <mean>0.0</mean>
+              <stddev>2e-4</stddev>
+              <bias_mean>0.0000075</bias_mean>
+              <bias_stddev>0.0000008</bias_stddev>
+            </noise>
           </y>
           <z>
-<!--            <noise type="gaussian">-->
-<!--              <mean>0.0</mean>-->
-<!--              <stddev>2e-4</stddev>-->
-<!--              <bias_mean>0.0000075</bias_mean>-->
-<!--              <bias_stddev>0.0000008</bias_stddev>-->
-<!--            </noise>-->
+            <noise type="gaussian">
+              <mean>0.0</mean>
+              <stddev>2e-4</stddev>
+              <bias_mean>0.0000075</bias_mean>
+              <bias_stddev>0.0000008</bias_stddev>
+            </noise>
           </z>
         </angular_velocity>
         <linear_acceleration>
           <x>
-<!--            <noise type="gaussian">-->
-<!--              <mean>0.0</mean>-->
-<!--              <stddev>1.7e-2</stddev>-->
-<!--              <bias_mean>0.1</bias_mean>-->
-<!--              <bias_stddev>0.001</bias_stddev>-->
-<!--            </noise>-->
+            <noise type="gaussian">
+              <mean>0.0</mean>
+              <stddev>1.7e-2</stddev>
+              <bias_mean>0.1</bias_mean>
+              <bias_stddev>0.001</bias_stddev>
+            </noise>
           </x>
           <y>
-<!--            <noise type="gaussian">-->
-<!--              <mean>0.0</mean>-->
-<!--              <stddev>1.7e-2</stddev>-->
-<!--              <bias_mean>0.1</bias_mean>-->
-<!--              <bias_stddev>0.001</bias_stddev>-->
-<!--            </noise>-->
+            <noise type="gaussian">
+              <mean>0.0</mean>
+              <stddev>1.7e-2</stddev>
+              <bias_mean>0.1</bias_mean>
+              <bias_stddev>0.001</bias_stddev>
+            </noise>
           </y>
           <z>
-<!--            <noise type="gaussian">-->
-<!--              <mean>0.0</mean>-->
-<!--              <stddev>1.7e-2</stddev>-->
-<!--              <bias_mean>0.1</bias_mean>-->
-<!--              <bias_stddev>0.001</bias_stddev>-->
-<!--            </noise>-->
+            <noise type="gaussian">
+              <mean>0.0</mean>
+              <stddev>1.7e-2</stddev>
+              <bias_mean>0.1</bias_mean>
+              <bias_stddev>0.001</bias_stddev>
+            </noise>
           </z>
         </linear_acceleration>
