Commit message: Add Gazebo Playground

File: descriptions/unitree/go2_description/xacro/gazebo.xacro (robot description, xacro)
@@ -1,170 +1,201 @@
 <?xml version="1.0"?>
 <robot xmlns:xacro="http://www.ros.org/wiki/xacro">
-	<ros2_control name="GazeboSystem" type="system">
-		<hardware>
-			<plugin>gz_ros2_control/GazeboSimSystem</plugin>
-		</hardware>
-		<joint name="FR_hip_joint">
-			<command_interface name="effort" initial_value="0.0"/>
-			<state_interface name="position"/>
-			<state_interface name="velocity"/>
-			<state_interface name="effort"/>
-		</joint>
-		<joint name="FR_thigh_joint">
-			<command_interface name="effort" initial_value="0.0"/>
-			<state_interface name="position"/>
-			<state_interface name="velocity"/>
-			<state_interface name="effort"/>
-		</joint>
-		<joint name="FR_calf_joint">
-			<command_interface name="effort" initial_value="0.0"/>
-			<state_interface name="position"/>
-			<state_interface name="velocity"/>
-			<state_interface name="effort"/>
-		</joint>
-		<joint name="FL_hip_joint">
-			<command_interface name="effort" initial_value="0.0"/>
-			<state_interface name="position"/>
-			<state_interface name="velocity"/>
-			<state_interface name="effort"/>
-		</joint>
-		<joint name="FL_thigh_joint">
-			<command_interface name="effort" initial_value="0.0"/>
-			<state_interface name="position"/>
-			<state_interface name="velocity"/>
-			<state_interface name="effort"/>
-		</joint>
-		<joint name="FL_calf_joint">
-			<command_interface name="effort" initial_value="0.0"/>
-			<state_interface name="position"/>
-			<state_interface name="velocity"/>
-			<state_interface name="effort"/>
-		</joint>
-		<joint name="RR_hip_joint">
-			<command_interface name="effort" initial_value="0.0"/>
-			<state_interface name="position"/>
-			<state_interface name="velocity"/>
-			<state_interface name="effort"/>
-		</joint>
-		<joint name="RR_thigh_joint">
-			<command_interface name="effort" initial_value="0.0"/>
-			<state_interface name="position"/>
-			<state_interface name="velocity"/>
-			<state_interface name="effort"/>
-		</joint>
-		<joint name="RR_calf_joint">
-			<command_interface name="effort" initial_value="0.0"/>
-			<state_interface name="position"/>
-			<state_interface name="velocity"/>
-			<state_interface name="effort"/>
-		</joint>
-		<joint name="RL_hip_joint">
-			<command_interface name="effort" initial_value="0.0"/>
-			<state_interface name="position"/>
-			<state_interface name="velocity"/>
-			<state_interface name="effort"/>
-		</joint>
-		<joint name="RL_thigh_joint">
-			<command_interface name="effort" initial_value="0.0"/>
-			<state_interface name="position"/>
-			<state_interface name="velocity"/>
-			<state_interface name="effort"/>
-		</joint>
-		<joint name="RL_calf_joint">
-			<command_interface name="effort" initial_value="0.0"/>
-			<state_interface name="position"/>
-			<state_interface name="velocity"/>
-			<state_interface name="effort"/>
-		</joint>
-		<sensor name="imu_sensor">
-			<state_interface name="orientation.x"/>
-			<state_interface name="orientation.y"/>
-			<state_interface name="orientation.z"/>
-			<state_interface name="orientation.w"/>
-			<state_interface name="angular_velocity.x"/>
-			<state_interface name="angular_velocity.y"/>
-			<state_interface name="angular_velocity.z"/>
-			<state_interface name="linear_acceleration.x"/>
-			<state_interface name="linear_acceleration.y"/>
-			<state_interface name="linear_acceleration.z"/>
-		</sensor>
-	</ros2_control>
-	<gazebo>
-		<plugin filename="gz_ros2_control-system" name="gz_ros2_control::GazeboSimROS2ControlPlugin">
-			<parameters>$(find go2_description)/config/gazebo.yaml</parameters>
-		</plugin>
-		<plugin filename="gz-sim-imu-system"
-						name="gz::sim::systems::Imu">
-		</plugin>
-	</gazebo>
-	<gazebo reference="trunk">
-		<mu1>0.6</mu1>
-		<mu2>0.6</mu2>
-		<self_collide>1</self_collide>
-	</gazebo>
-	<gazebo reference="imu_link">
-		<sensor name="imu_sensor" type="imu">
-			<always_on>1</always_on>
-			<update_rate>500</update_rate>
-			<visualize>true</visualize>
-			<topic>imu</topic>
-			<imu>
-				<angular_velocity>
-					<x>
-						<noise type="gaussian">
-							<mean>0.0</mean>
-							<stddev>2e-4</stddev>
-							<bias_mean>0.0000075</bias_mean>
-							<bias_stddev>0.0000008</bias_stddev>
-						</noise>
-					</x>
-					<y>
-						<noise type="gaussian">
-							<mean>0.0</mean>
-							<stddev>2e-4</stddev>
-							<bias_mean>0.0000075</bias_mean>
-							<bias_stddev>0.0000008</bias_stddev>
-						</noise>
-					</y>
-					<z>
-						<noise type="gaussian">
-							<mean>0.0</mean>
-							<stddev>2e-4</stddev>
-							<bias_mean>0.0000075</bias_mean>
-							<bias_stddev>0.0000008</bias_stddev>
-						</noise>
-					</z>
-				</angular_velocity>
-				<linear_acceleration>
-					<x>
-						<noise type="gaussian">
-							<mean>0.0</mean>
-							<stddev>1.7e-2</stddev>
-							<bias_mean>0.1</bias_mean>
-							<bias_stddev>0.001</bias_stddev>
-						</noise>
-					</x>
-					<y>
-						<noise type="gaussian">
-							<mean>0.0</mean>
-							<stddev>1.7e-2</stddev>
-							<bias_mean>0.1</bias_mean>
-							<bias_stddev>0.001</bias_stddev>
-						</noise>
-					</y>
-					<z>
-						<noise type="gaussian">
-							<mean>0.0</mean>
-							<stddev>1.7e-2</stddev>
-							<bias_mean>0.1</bias_mean>
-							<bias_stddev>0.001</bias_stddev>
-						</noise>
-					</z>
-				</linear_acceleration>
-			</imu>
-		</sensor>
-	</gazebo>
-	<gazebo reference="imu_joint">
-		<disableFixedJointLumping>true</disableFixedJointLumping>
-	</gazebo>
+    <ros2_control name="GazeboSystem" type="system">
+        <hardware>
+            <plugin>gz_ros2_control/GazeboSimSystem</plugin>
+        </hardware>
+        <joint name="FR_hip_joint">
+            <command_interface name="effort" initial_value="0.0"/>
+            <state_interface name="position"/>
+            <state_interface name="velocity"/>
+            <state_interface name="effort"/>
+        </joint>
+        <joint name="FR_thigh_joint">
+            <command_interface name="effort" initial_value="0.0"/>
+            <state_interface name="position"/>
+            <state_interface name="velocity"/>
+            <state_interface name="effort"/>
+        </joint>
+        <joint name="FR_calf_joint">
+            <command_interface name="effort" initial_value="0.0"/>
+            <state_interface name="position"/>
+            <state_interface name="velocity"/>
+            <state_interface name="effort"/>
+        </joint>
+        <joint name="FL_hip_joint">
+            <command_interface name="effort" initial_value="0.0"/>
+            <state_interface name="position"/>
+            <state_interface name="velocity"/>
+            <state_interface name="effort"/>
+        </joint>
+        <joint name="FL_thigh_joint">
+            <command_interface name="effort" initial_value="0.0"/>
+            <state_interface name="position"/>
+            <state_interface name="velocity"/>
+            <state_interface name="effort"/>
+        </joint>
+        <joint name="FL_calf_joint">
+            <command_interface name="effort" initial_value="0.0"/>
+            <state_interface name="position"/>
+            <state_interface name="velocity"/>
+            <state_interface name="effort"/>
+        </joint>
+        <joint name="RR_hip_joint">
+            <command_interface name="effort" initial_value="0.0"/>
+            <state_interface name="position"/>
+            <state_interface name="velocity"/>
+            <state_interface name="effort"/>
+        </joint>
+        <joint name="RR_thigh_joint">
+            <command_interface name="effort" initial_value="0.0"/>
+            <state_interface name="position"/>
+            <state_interface name="velocity"/>
+            <state_interface name="effort"/>
+        </joint>
+        <joint name="RR_calf_joint">
+            <command_interface name="effort" initial_value="0.0"/>
+            <state_interface name="position"/>
+            <state_interface name="velocity"/>
+            <state_interface name="effort"/>
+        </joint>
+        <joint name="RL_hip_joint">
+            <command_interface name="effort" initial_value="0.0"/>
+            <state_interface name="position"/>
+            <state_interface name="velocity"/>
+            <state_interface name="effort"/>
+        </joint>
+        <joint name="RL_thigh_joint">
+            <command_interface name="effort" initial_value="0.0"/>
+            <state_interface name="position"/>
+            <state_interface name="velocity"/>
+            <state_interface name="effort"/>
+        </joint>
+        <joint name="RL_calf_joint">
+            <command_interface name="effort" initial_value="0.0"/>
+            <state_interface name="position"/>
+            <state_interface name="velocity"/>
+            <state_interface name="effort"/>
+        </joint>
+        <sensor name="imu_sensor">
+            <state_interface name="orientation.x"/>
+            <state_interface name="orientation.y"/>
+            <state_interface name="orientation.z"/>
+            <state_interface name="orientation.w"/>
+            <state_interface name="angular_velocity.x"/>
+            <state_interface name="angular_velocity.y"/>
+            <state_interface name="angular_velocity.z"/>
+            <state_interface name="linear_acceleration.x"/>
+            <state_interface name="linear_acceleration.y"/>
+            <state_interface name="linear_acceleration.z"/>
+        </sensor>
+    </ros2_control>
+    <gazebo>
+        <plugin filename="gz_ros2_control-system" name="gz_ros2_control::GazeboSimROS2ControlPlugin">
+            <parameters>$(find go2_description)/config/gazebo.yaml</parameters>
+        </plugin>
+        <plugin filename="gz-sim-imu-system"
+                name="gz::sim::systems::Imu">
+        </plugin>
+    </gazebo>
+    <gazebo reference="trunk">
+        <mu1>0.6</mu1>
+        <mu2>0.6</mu2>
+        <self_collide>1</self_collide>
+    </gazebo>
+    <gazebo reference="imu_link">
+        <sensor name="imu_sensor" type="imu">
+            <always_on>1</always_on>
+            <update_rate>500</update_rate>
+            <visualize>true</visualize>
+            <topic>imu</topic>
+            <imu>
+                <angular_velocity>
+                    <x>
+                        <noise type="gaussian">
+                            <mean>0.0</mean>
+                            <stddev>2e-4</stddev>
+                            <bias_mean>0.0000075</bias_mean>
+                            <bias_stddev>0.0000008</bias_stddev>
+                        </noise>
+                    </x>
+                    <y>
+                        <noise type="gaussian">
+                            <mean>0.0</mean>
+                            <stddev>2e-4</stddev>
+                            <bias_mean>0.0000075</bias_mean>
+                            <bias_stddev>0.0000008</bias_stddev>
+                        </noise>
+                    </y>
+                    <z>
+                        <noise type="gaussian">
+                            <mean>0.0</mean>
+                            <stddev>2e-4</stddev>
+                            <bias_mean>0.0000075</bias_mean>
+                            <bias_stddev>0.0000008</bias_stddev>
+                        </noise>
+                    </z>
+                </angular_velocity>
+                <linear_acceleration>
+                    <x>
+                        <noise type="gaussian">
+                            <mean>0.0</mean>
+                            <stddev>1.7e-2</stddev>
+                            <bias_mean>0.1</bias_mean>
+                            <bias_stddev>0.001</bias_stddev>
+                        </noise>
+                    </x>
+                    <y>
+                        <noise type="gaussian">
+                            <mean>0.0</mean>
+                            <stddev>1.7e-2</stddev>
+                            <bias_mean>0.1</bias_mean>
+                            <bias_stddev>0.001</bias_stddev>
+                        </noise>
+                    </y>
+                    <z>
+                        <noise type="gaussian">
+                            <mean>0.0</mean>
+                            <stddev>1.7e-2</stddev>
+                            <bias_mean>0.1</bias_mean>
+                            <bias_stddev>0.001</bias_stddev>
+                        </noise>
+                    </z>
+                </linear_acceleration>
+            </imu>
+        </sensor>
+    </gazebo>
+    <gazebo reference="imu_joint">
+        <disableFixedJointLumping>true</disableFixedJointLumping>
+    </gazebo>
+	<xacro:if value="$(arg EXTERNAL_SENSORS)">
+        <gazebo reference="front_camera">
+            <sensor name="front_camera" type="camera">
+                <camera>
+                    <horizontal_fov>2.094</horizontal_fov>
+                    <image>
+                        <width>1280</width>
+                        <height>720</height>
+                    </image>
+                    <clip>
+                        <near>0.1</near>
+                        <far>15</far>
+                    </clip>
+                    <noise>
+                        <type>gaussian</type>
+                        <!-- Noise is sampled independently per pixel on each frame.
+                            That pixel's noise value is added to each of its color
+                            channels, which at that point lie in the range [0,1]. -->
+                        <mean>0.0</mean>
+                        <stddev>0.007</stddev>
+                    </noise>
+                    <optical_frame_id>front_camera</optical_frame_id>
+                    <camera_info_topic>camera/camera_info</camera_info_topic>
+                </camera>
+                <always_on>true</always_on>
+                <update_rate>15</update_rate>
+                <visualize>true</visualize>
+                <topic>camera/image</topic>
+            </sensor>
+        </gazebo>
+	</xacro:if>
 </robot>

File: descriptions/unitree/go2_description/xacro/robot.xacro (robot description, xacro)
@@ -109,30 +109,11 @@
 		</collision>
 	</link>
-	<!--
-	<joint name="load_joint" type="fixed">
-			<parent link="trunk"/>
-			<child link="load_link"/>
-			<origin rpy="0 0 0" xyz="0 0 0"/>
+	<joint name="front_camera_joint" type="fixed">
+		<parent link="trunk"/>
+		<child link="front_camera"/>
+		<origin rpy="0 0 0" xyz="0.32715 0 0.04297"/>
 	</joint>
-	<link name="load_link">
-			<inertial>
-					<mass value="5"/>
-					<origin rpy="0 0 0" xyz="0 0 0"/>
-					<inertia ixx="0.01" ixy="0" ixz="0" iyy="0.01" iyz="0" izz="0.01"/>
-			</inertial>
-			<visual>
-					<origin rpy="0 0 0" xyz="0 0 0.2"/>
-					<geometry>
-							<box size="0.5 0.3 0.2"/>
-					</geometry>
-			</visual>
-			<collision>
-					<origin rpy="0 0 0" xyz="0 0 0"/>
-					<geometry>
-							<box size=".001 .001 .001"/>
-					</geometry>
-			</collision>
+	<link name="front_camera">
 	</link>
--->
 	<xacro:leg name="FR" mirror="-1" mirror_dae="False" front_hind="1" front_hind_dae="True"/>
 	<xacro:leg name="FL" mirror="1" mirror_dae="True" front_hind="1" front_hind_dae="True"/>
