Commit message: add lidar for deep robotics lite3

File: descriptions/deep_robotics/lite3_description/xacro/gazebo.xacro (robot description, xacro)
@@ -1,10 +1,15 @@
 <?xml version="1.0"?>
 <robot xmlns:xacro="http://www.ros.org/wiki/xacro">
+  <xacro:include filename="$(find gz_quadruped_hardware)/xacro/foot_force_sensor.xacro"/>
   <ros2_control name="GazeboSystem" type="system">
     <hardware>
-      <plugin>gz_ros2_control/GazeboSimSystem</plugin>
+      <plugin>gz_quadruped_hardware/GazeboSimSystem</plugin>
     </hardware>
     <joint name="FR_HipX">
-      <command_interface name="effort" initial_value="0.0"/>
+      <command_interface name="position"/>
+      <command_interface name="velocity"/>
+      <command_interface name="effort"/>
+      <command_interface name="kp"/>
+      <command_interface name="kd"/>
       <state_interface name="position"/>
       <state_interface name="velocity"/>
@@ -12,5 +17,9 @@
     </joint>
     <joint name="FR_HipY">
-      <command_interface name="effort" initial_value="0.0"/>
+      <command_interface name="position"/>
+      <command_interface name="velocity"/>
+      <command_interface name="effort"/>
+      <command_interface name="kp"/>
+      <command_interface name="kd"/>
       <state_interface name="position"/>
       <state_interface name="velocity"/>
@@ -18,5 +27,9 @@
     </joint>
     <joint name="FR_Knee">
-      <command_interface name="effort" initial_value="0.0"/>
+      <command_interface name="position"/>
+      <command_interface name="velocity"/>
+      <command_interface name="effort"/>
+      <command_interface name="kp"/>
+      <command_interface name="kd"/>
       <state_interface name="position"/>
       <state_interface name="velocity"/>
@@ -24,5 +37,9 @@
     </joint>
     <joint name="FL_HipX">
-      <command_interface name="effort" initial_value="0.0"/>
+      <command_interface name="position"/>
+      <command_interface name="velocity"/>
+      <command_interface name="effort"/>
+      <command_interface name="kp"/>
+      <command_interface name="kd"/>
       <state_interface name="position"/>
       <state_interface name="velocity"/>
@@ -30,5 +47,9 @@
     </joint>
     <joint name="FL_HipY">
-      <command_interface name="effort" initial_value="0.0"/>
+      <command_interface name="position"/>
+      <command_interface name="velocity"/>
+      <command_interface name="effort"/>
+      <command_interface name="kp"/>
+      <command_interface name="kd"/>
       <state_interface name="position"/>
       <state_interface name="velocity"/>
@@ -36,5 +57,9 @@
     </joint>
     <joint name="FL_Knee">
-      <command_interface name="effort" initial_value="0.0"/>
+      <command_interface name="position"/>
+      <command_interface name="velocity"/>
+      <command_interface name="effort"/>
+      <command_interface name="kp"/>
+      <command_interface name="kd"/>
       <state_interface name="position"/>
       <state_interface name="velocity"/>
@@ -42,5 +67,9 @@
     </joint>
     <joint name="HR_HipX">
-      <command_interface name="effort" initial_value="0.0"/>
+      <command_interface name="position"/>
+      <command_interface name="velocity"/>
+      <command_interface name="effort"/>
+      <command_interface name="kp"/>
+      <command_interface name="kd"/>
       <state_interface name="position"/>
       <state_interface name="velocity"/>
@@ -48,5 +77,9 @@
     </joint>
     <joint name="HR_HipY">
-      <command_interface name="effort" initial_value="0.0"/>
+      <command_interface name="position"/>
+      <command_interface name="velocity"/>
+      <command_interface name="effort"/>
+      <command_interface name="kp"/>
+      <command_interface name="kd"/>
       <state_interface name="position"/>
       <state_interface name="velocity"/>
@@ -54,5 +87,9 @@
     </joint>
     <joint name="HR_Knee">
-      <command_interface name="effort" initial_value="0.0"/>
+      <command_interface name="position"/>
+      <command_interface name="velocity"/>
+      <command_interface name="effort"/>
+      <command_interface name="kp"/>
+      <command_interface name="kd"/>
       <state_interface name="position"/>
       <state_interface name="velocity"/>
@@ -60,5 +97,9 @@
     </joint>
     <joint name="HL_HipX">
-      <command_interface name="effort" initial_value="0.0"/>
+      <command_interface name="position"/>
+      <command_interface name="velocity"/>
+      <command_interface name="effort"/>
+      <command_interface name="kp"/>
+      <command_interface name="kd"/>
       <state_interface name="position"/>
       <state_interface name="velocity"/>
@@ -66,5 +107,9 @@
     </joint>
     <joint name="HL_HipY">
-      <command_interface name="effort" initial_value="0.0"/>
+      <command_interface name="position"/>
+      <command_interface name="velocity"/>
+      <command_interface name="effort"/>
+      <command_interface name="kp"/>
+      <command_interface name="kd"/>
       <state_interface name="position"/>
       <state_interface name="velocity"/>
@@ -72,5 +117,9 @@
     </joint>
     <joint name="HL_Knee">
-      <command_interface name="effort" initial_value="0.0"/>
+      <command_interface name="position"/>
+      <command_interface name="velocity"/>
+      <command_interface name="effort"/>
+      <command_interface name="kp"/>
+      <command_interface name="kd"/>
       <state_interface name="position"/>
       <state_interface name="velocity"/>
@@ -89,7 +138,13 @@
       <state_interface name="linear_acceleration.z"/>
     </sensor>
+    <sensor name="foot_force">
+      <state_interface name="FR_foot_force"/>
+      <state_interface name="FL_foot_force"/>
+      <state_interface name="HR_foot_force"/>
+      <state_interface name="HL_foot_force"/>
+    </sensor>
   </ros2_control>
   <gazebo>
-    <plugin filename="gz_ros2_control-system" name="gz_ros2_control::GazeboSimROS2ControlPlugin">
+    <plugin filename="gz_quadruped_hardware-system" name="gz_quadruped_hardware::GazeboSimQuadrupedPlugin">
       <parameters>$(find lite3_description)/config/gazebo.yaml</parameters>
     </plugin>
@@ -97,4 +152,15 @@
             name="gz::sim::systems::Imu">
     </plugin>
+    <plugin filename="gz-sim-forcetorque-system" name="gz::sim::systems::ForceTorque"/>
+    <!--    <plugin filename="gz-sim-odometry-publisher-system"-->
+    <!--            name="gz::sim::systems::OdometryPublisher">-->
+    <!--      <odom_frame>odom</odom_frame>-->
+    <!--      <robot_base_frame>base</robot_base_frame>-->
+    <!--      <odom_publish_frequency>1000</odom_publish_frequency>-->
+    <!--      <odom_topic>odom</odom_topic>-->
+    <!--      <dimensions>3</dimensions>-->
+    <!--      <odom_covariance_topic>odom_with_covariance</odom_covariance_topic>-->
+    <!--      <tf_topic>tf</tf_topic>-->
+    <!--    </plugin>-->
   </gazebo>
   <gazebo reference="trunk">
@@ -112,52 +178,52 @@
         <angular_velocity>
           <x>
-<!--            <noise type="gaussian">-->
-<!--              <mean>0.0</mean>-->
-<!--              <stddev>2e-4</stddev>-->
-<!--              <bias_mean>0.0000075</bias_mean>-->
-<!--              <bias_stddev>0.0000008</bias_stddev>-->
-<!--            </noise>-->
+            <noise type="gaussian">
+              <mean>0.0</mean>
+              <stddev>2e-4</stddev>
+              <bias_mean>0.0000075</bias_mean>
+              <bias_stddev>0.0000008</bias_stddev>
+            </noise>
           </x>
           <y>
-<!--            <noise type="gaussian">-->
-<!--              <mean>0.0</mean>-->
-<!--              <stddev>2e-4</stddev>-->
-<!--              <bias_mean>0.0000075</bias_mean>-->
-<!--              <bias_stddev>0.0000008</bias_stddev>-->
-<!--            </noise>-->
+            <noise type="gaussian">
+              <mean>0.0</mean>
+              <stddev>2e-4</stddev>
+              <bias_mean>0.0000075</bias_mean>
+              <bias_stddev>0.0000008</bias_stddev>
+            </noise>
           </y>
           <z>
-<!--            <noise type="gaussian">-->
-<!--              <mean>0.0</mean>-->
-<!--              <stddev>2e-4</stddev>-->
-<!--              <bias_mean>0.0000075</bias_mean>-->
-<!--              <bias_stddev>0.0000008</bias_stddev>-->
-<!--            </noise>-->
+            <noise type="gaussian">
+              <mean>0.0</mean>
+              <stddev>2e-4</stddev>
+              <bias_mean>0.0000075</bias_mean>
+              <bias_stddev>0.0000008</bias_stddev>
+            </noise>
           </z>
         </angular_velocity>
         <linear_acceleration>
           <x>
-<!--            <noise type="gaussian">-->
-<!--              <mean>0.0</mean>-->
-<!--              <stddev>1.7e-2</stddev>-->
-<!--              <bias_mean>0.1</bias_mean>-->
-<!--              <bias_stddev>0.001</bias_stddev>-->
-<!--            </noise>-->
+            <noise type="gaussian">
+              <mean>0.0</mean>
+              <stddev>1.7e-2</stddev>
+              <bias_mean>0.1</bias_mean>
+              <bias_stddev>0.001</bias_stddev>
+            </noise>
           </x>
           <y>
-<!--            <noise type="gaussian">-->
-<!--              <mean>0.0</mean>-->
-<!--              <stddev>1.7e-2</stddev>-->
-<!--              <bias_mean>0.1</bias_mean>-->
-<!--              <bias_stddev>0.001</bias_stddev>-->
-<!--            </noise>-->
+            <noise type="gaussian">
+              <mean>0.0</mean>
+              <stddev>1.7e-2</stddev>
+              <bias_mean>0.1</bias_mean>
+              <bias_stddev>0.001</bias_stddev>
+            </noise>
           </y>
           <z>
-<!--            <noise type="gaussian">-->
-<!--              <mean>0.0</mean>-->
-<!--              <stddev>1.7e-2</stddev>-->
-<!--              <bias_mean>0.1</bias_mean>-->
-<!--              <bias_stddev>0.001</bias_stddev>-->
-<!--            </noise>-->
+            <noise type="gaussian">
+              <mean>0.0</mean>
+              <stddev>1.7e-2</stddev>
+              <bias_mean>0.1</bias_mean>
+              <bias_stddev>0.001</bias_stddev>
+            </noise>
           </z>
         </linear_acceleration>
@@ -168,3 +234,18 @@
     <disableFixedJointLumping>true</disableFixedJointLumping>
   </gazebo>
+  <xacro:foot_force_sensor name="FL" suffix="Ankle"/>
+  <xacro:foot_force_sensor name="HL" suffix="Ankle"/>
+  <xacro:foot_force_sensor name="FR" suffix="Ankle"/>
+  <xacro:foot_force_sensor name="HR" suffix="Ankle"/>
+  <xacro:arg name="EXTERNAL_SENSORS" default="false"/>
+  <xacro:if value="$(arg EXTERNAL_SENSORS)">
+    <xacro:include filename="$(find gz_quadruped_playground)/models/D435/model.xacro"/>
+    <xacro:include filename="$(find gz_quadruped_playground)/models/Lidar3DV1/model.xacro"/>
+    <xacro:d435 camID="1" name="d435">
+      <origin rpy="0 0.1 0" xyz="0.23 0 0.06"/>
+    </xacro:d435>
+    <xacro:Lidar3D vertical="16" name="lslidar">
+      <origin rpy="0 0 0" xyz="0.163 0 0.058"/>
+    </xacro:Lidar3D>
+  </xacro:if>
 </robot>

File: descriptions/deep_robotics/lite3_description/xacro/robot.xacro (robot description, xacro)
@@ -1,6 +1,6 @@
 <?xml version="1.0"?>
 <robot name="lite3" xmlns:xacro="http://www.ros.org/wiki/xacro">
-  <xacro:include filename="$(find lite3_description)/xacro/body.xacro"/>
-  <xacro:include filename="$(find lite3_description)/xacro/transmission.xacro"/>
+  <xacro:include filename="$(find lite3_description)/xacro/const.xacro"/>
+  <xacro:include filename="$(find lite3_description)/xacro/leg.xacro"/>
   <xacro:arg name="GAZEBO" default="false"/>
   <xacro:arg name="CLASSIC" default="false"/>
@@ -16,3 +16,63 @@
     <xacro:include filename="$(find lite3_description)/xacro/ros2_control.xacro"/>
   </xacro:unless>
+  <link name="base">
+    <visual>
+      <origin rpy="0 0 0" xyz="0 0 0"/>
+      <geometry>
+        <box size="0.001 0.001 0.001"/>
+      </geometry>
+    </visual>
+  </link>
+  <joint name="floating_base" type="fixed">
+    <origin rpy="0 0 0" xyz="0 0 0"/>
+    <parent link="base"/>
+    <child link="TORSO"/>
+  </joint>
+  <link name="TORSO">
+    <visual>
+      <origin rpy="0 0 3.1416" xyz="0.0 0.0 0.0"/>
+      <geometry>
+        <mesh filename="file://$(find lite3_description)/meshes/Lite3.dae"/>
+      </geometry>
+    </visual>
+    <collision>
+      <geometry>
+        <box size="0.35 0.184 0.08"/>
+      </geometry>
+    </collision>
+    <inertial>
+      <origin xyz="0.004098 -0.000663 -0.002069"/>
+      <mass value="4.130"/>
+      <inertia ixx="0.016982120" ixy="2.1294E-05" ixz="6.0763E-05" iyy="0.030466501" iyz="1.7968E-05"
+               izz="0.042609956"/>
+    </inertial>
+  </link>
+  <joint name="imu_joint" type="fixed">
+    <parent link="TORSO"/>
+    <child link="imu_link"/>
+    <origin rpy="0 0 0" xyz="0 0 0"/>
+  </joint>
+  <link name="imu_link">
+    <inertial>
+      <mass value="0.001"/>
+      <origin rpy="0 0 0" xyz="0 0 0"/>
+      <inertia ixx="0.0001" ixy="0" ixz="0" iyy="0.0001" iyz="0" izz="0.0001"/>
+    </inertial>
+    <visual>
+      <origin rpy="0 0 0" xyz="0 0 0"/>
+      <geometry>
+        <box size="0.001 0.001 0.001"/>
+      </geometry>
+    </visual>
+    <collision>
+      <origin rpy="0 0 0" xyz="0 0 0"/>
+      <geometry>
+        <box size=".001 .001 .001"/>
+      </geometry>
+    </collision>
+  </link>
+  <xacro:leg name="FR" mirror="-1" mirror_dae="False" front_hind="1" front_hind_dae="True"/>
+  <xacro:leg name="FL" mirror="1" mirror_dae="True" front_hind="1" front_hind_dae="True"/>
+  <xacro:leg name="HR" mirror="-1" mirror_dae="False" front_hind="-1" front_hind_dae="False"/>
+  <xacro:leg name="HL" mirror="1" mirror_dae="True" front_hind="-1" front_hind_dae="False"/>
 </robot>

File: descriptions/deep_robotics/lite3_description/xacro/transmission.xacro (robot description, xacro)
@@ -1,115 +1,32 @@
 <?xml version="1.0"?>
 <robot xmlns:xacro="http://www.ros.org/wiki/xacro">
-  <!-- FL transmissions -->
-  <transmission name="FL_HipX_tran">
-    <type>transmission_interface/SimpleTransmission</type>
-    <joint name="FL_HipX">
-      <hardwareInterface>hardware_interface/EffortJointInterface</hardwareInterface>
-    </joint>
-    <actuator name="FL_HipX_motor">
-      <mechanicalReduction>1</mechanicalReduction>
-    </actuator>
-  </transmission>
-  <transmission name="FL_HipY_tran">
-    <type>transmission_interface/SimpleTransmission</type>
-    <joint name="FL_HipY">
-      <hardwareInterface>hardware_interface/EffortJointInterface</hardwareInterface>
-    </joint>
-    <actuator name="FL_HipY_motor">
-      <mechanicalReduction>1</mechanicalReduction>
-    </actuator>
-  </transmission>
-  <transmission name="FL_Knee_tran">
-    <type>transmission_interface/SimpleTransmission</type>
-    <joint name="FL_Knee">
-      <hardwareInterface>hardware_interface/EffortJointInterface</hardwareInterface>
-    </joint>
-    <actuator name="FL_Knee_motor">
-      <mechanicalReduction>1</mechanicalReduction>
-    </actuator>
-  </transmission>
-  <!-- FR transmissions -->
-  <transmission name="FR_HipX_tran">
-    <type>transmission_interface/SimpleTransmission</type>
-    <joint name="FR_HipX">
-      <hardwareInterface>hardware_interface/EffortJointInterface</hardwareInterface>
-    </joint>
-    <actuator name="FR_HipX_motor">
-      <mechanicalReduction>1</mechanicalReduction>
-    </actuator>
-  </transmission>
-  <transmission name="FR_HipY_tran">
-    <type>transmission_interface/SimpleTransmission</type>
-    <joint name="FR_HipY">
-      <hardwareInterface>hardware_interface/EffortJointInterface</hardwareInterface>
-    </joint>
-    <actuator name="FR_HipY_motor">
-      <mechanicalReduction>1</mechanicalReduction>
-    </actuator>
-  </transmission>
-  <transmission name="FR_Knee_tran">
-    <type>transmission_interface/SimpleTransmission</type>
-    <joint name="FR_Knee">
-      <hardwareInterface>hardware_interface/EffortJointInterface</hardwareInterface>
-    </joint>
-    <actuator name="FR_Knee_motor">
-      <mechanicalReduction>1</mechanicalReduction>
-    </actuator>
-  </transmission>
-  <!-- HL transmissions -->
-  <transmission name="HL_HipX_tran">
-    <type>transmission_interface/SimpleTransmission</type>
-    <joint name="HL_HipX">
-      <hardwareInterface>hardware_interface/EffortJointInterface</hardwareInterface>
-    </joint>
-    <actuator name="HL_HipX_motor">
-      <mechanicalReduction>1</mechanicalReduction>
-    </actuator>
-  </transmission>
-  <transmission name="HL_HipY_tran">
-    <type>transmission_interface/SimpleTransmission</type>
-    <joint name="HL_HipY">
-      <hardwareInterface>hardware_interface/EffortJointInterface</hardwareInterface>
-    </joint>
-    <actuator name="HL_HipY_motor">
-      <mechanicalReduction>1</mechanicalReduction>
-    </actuator>
-  </transmission>
-  <transmission name="HL_Knee_tran">
-    <type>transmission_interface/SimpleTransmission</type>
-    <joint name="HL_Knee">
-      <hardwareInterface>hardware_interface/EffortJointInterface</hardwareInterface>
-    </joint>
-    <actuator name="HL_Knee_motor">
-      <mechanicalReduction>1</mechanicalReduction>
-    </actuator>
-  </transmission>
-  <!-- HR transmissions -->
-  <transmission name="HR_HipX_tran">
-    <type>transmission_interface/SimpleTransmission</type>
-    <joint name="HR_HipX">
-      <hardwareInterface>hardware_interface/EffortJointInterface</hardwareInterface>
-    </joint>
-    <actuator name="HR_HipX_motor">
-      <mechanicalReduction>1</mechanicalReduction>
-    </actuator>
-  </transmission>
-  <transmission name="HR_HipY_tran">
-    <type>transmission_interface/SimpleTransmission</type>
-    <joint name="HR_HipY">
-      <hardwareInterface>hardware_interface/EffortJointInterface</hardwareInterface>
-    </joint>
-    <actuator name="HR_HipY_motor">
-      <mechanicalReduction>1</mechanicalReduction>
-    </actuator>
-  </transmission>
-  <transmission name="HR_Knee_tran">
-    <type>transmission_interface/SimpleTransmission</type>
-    <joint name="HR_Knee">
-      <hardwareInterface>hardware_interface/EffortJointInterface</hardwareInterface>
-    </joint>
-    <actuator name="HR_Knee_motor">
-      <mechanicalReduction>1</mechanicalReduction>
-    </actuator>
-  </transmission>
+  <xacro:macro name="leg_transmission" params="name">
+    <transmission name="${name}_HipX_tran">
+      <type>transmission_interface/SimpleTransmission</type>
+      <joint name="${name}_HipX">
+        <hardwareInterface>hardware_interface/EffortJointInterface</hardwareInterface>
+      </joint>
+      <actuator name="${name}_HipX_motor">
+        <mechanicalReduction>1</mechanicalReduction>
+      </actuator>
+    </transmission>
+    <transmission name="{name}_HipY_tran">
+      <type>transmission_interface/SimpleTransmission</type>
+      <joint name="{name}_HipY">
+        <hardwareInterface>hardware_interface/EffortJointInterface</hardwareInterface>
+      </joint>
+      <actuator name="{name}_HipY_motor">
+        <mechanicalReduction>1</mechanicalReduction>
+      </actuator>
+    </transmission>
+    <transmission name="{name}_Knee_tran">
+      <type>transmission_interface/SimpleTransmission</type>
+      <joint name="{name}_Knee">
+        <hardwareInterface>hardware_interface/EffortJointInterface</hardwareInterface>
+      </joint>
+      <actuator name="{name}_Knee_motor">
+        <mechanicalReduction>1</mechanicalReduction>
+      </actuator>
+    </transmission>
+  </xacro:macro>
 </robot>

File: descriptions/unitree/go2_description/xacro/const.xacro (robot description, xacro)
@@ -40,5 +40,5 @@
 	<!-- joint limits -->
 	<xacro:property name="damping" value="0.0"/>
-	<xacro:property name="friction" value="0.0"/>
+	<xacro:property name="friction" value="0.01"/>
 	<xacro:property name="hip_position_max" value="1.0472"/>
 	<xacro:property name="hip_position_min" value="-1.0472"/>

File: descriptions/unitree/go2_description/xacro/gazebo.xacro (robot description, xacro)
@@ -153,14 +153,4 @@
     </plugin>
     <plugin filename="gz-sim-forcetorque-system" name="gz::sim::systems::ForceTorque"/>
-    <plugin filename="gz-sim-odometry-publisher-system"
-            name="gz::sim::systems::OdometryPublisher">
-      <odom_frame>odom</odom_frame>
-      <robot_base_frame>base</robot_base_frame>
-      <odom_publish_frequency>1000</odom_publish_frequency>
-      <odom_topic>odom</odom_topic>
-      <dimensions>3</dimensions>
-      <odom_covariance_topic>odom_with_covariance</odom_covariance_topic>
-      <tf_topic>tf</tf_topic>
-    </plugin>
   </gazebo>
   <gazebo reference="trunk">
@@ -234,8 +224,8 @@
     <disableFixedJointLumping>true</disableFixedJointLumping>
   </gazebo>
-  <xacro:foot_force_sensor name="FL"/>
-  <xacro:foot_force_sensor name="RL"/>
-  <xacro:foot_force_sensor name="FR"/>
-  <xacro:foot_force_sensor name="RR"/>
+  <xacro:foot_force_sensor name="FL" suffix="foot_fixed"/>
+  <xacro:foot_force_sensor name="RL" suffix="foot_fixed"/>
+  <xacro:foot_force_sensor name="FR" suffix="foot_fixed"/>
+  <xacro:foot_force_sensor name="RR" suffix="foot_fixed"/>
   <xacro:arg name="EXTERNAL_SENSORS" default="false"/>
   <xacro:if value="$(arg EXTERNAL_SENSORS)">

File: hardwares/gz_quadruped_hardware/xacro/foot_force_sensor.xacro (robot description, xacro)
@@ -1,6 +1,6 @@
 <?xml version="1.0"?>
 <robot xmlns:xacro="http://www.ros.org/wiki/xacro">
-  <xacro:macro name="foot_force_sensor" params="name">
-    <gazebo reference="${name}_foot_fixed">
+  <xacro:macro name="foot_force_sensor" params="name suffix">
+    <gazebo reference="${name}_${suffix}">
       <!-- Enable feedback for this joint -->
       <provide_feedback>true</provide_feedback>

File: libraries/gz_quadruped_playground/models/D435/model.xacro (robot description, xacro)
@@ -4,5 +4,5 @@
     <joint name="camera_joint_${name}" type="fixed">
       <xacro:insert_block name="origin"/>
-      <parent link="trunk"/>
+      <parent link="base"/>
       <child link="camera_${name}"/>
     </joint>
@@ -74,5 +74,5 @@
         </camera>
         <always_on>true</always_on>
-        <update_rate>15</update_rate>
+        <update_rate>30</update_rate>
         <visualize>true</visualize>
         <topic>rgbd_${name}</topic>
