Commit message: add ocs2 control for deep robotics

File: descriptions/deep_robotics/x30_description/urdf/robot.urdf (robot description, URDF)
Before this commit: robot X30, 17 links, 16 joints
Links:
- added link base; visual box size=0.001 0.001 0.001
- added link imu_link, mass 0.001; collision box size=.001 .001 .001; visual box size=0.001 0.001 0.001
- link FL_HIP: geometry visual mesh filename=file:///home/hiverlab/ros2_ws/install/x30_description/share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
- link FL_SHANK: geometry collision cylinder length=0.08 radius=0.022; collision cylinder length=0.1 radius=0.025
- link FL_THIGH: geometry collision cylinder length=0.25 radius=0.04; visual mesh filename=file:///home/hiverlab/ros2_ws/install/x30_description/share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
- link FR_HIP: geometry visual mesh filename=file:///home/hiverlab/ros2_ws/install/x30_description/share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
- link FR_SHANK: geometry collision cylinder length=0.08 radius=0.022; collision cylinder length=0.1 radius=0.025
- link FR_THIGH: geometry collision cylinder length=0.25 radius=0.04; visual mesh filename=file:///home/hiverlab/ros2_ws/install/x30_description/share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
- link HL_HIP: geometry visual mesh filename=file:///home/hiverlab/ros2_ws/install/x30_description/share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
- link HL_SHANK: geometry collision cylinder length=0.08 radius=0.022; collision cylinder length=0.1 radius=0.025
- link HL_THIGH: geometry collision cylinder length=0.25 radius=0.04; visual mesh filename=file:///home/hiverlab/ros2_ws/install/x30_description/share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
- link HR_HIP: geometry visual mesh filename=file:///home/hiverlab/ros2_ws/install/x30_description/share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
- link HR_SHANK: geometry collision cylinder length=0.08 radius=0.022; collision cylinder length=0.1 radius=0.025
- link HR_THIGH: geometry collision cylinder length=0.25 radius=0.04; visual mesh filename=file:///home/hiverlab/ros2_ws/install/x30_description/share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
- link TORSO: geometry collision box size=0.44 0.26 0.15; visual mesh filename=file:///home/hiverlab/ros2_ws/install/x30_description/share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
Joints:
- removed joint FL_HipX_joint
- removed joint FL_HipY_joint
- removed joint FL_Knee_joint
- removed joint FR_HipX_joint
- removed joint FR_HipY_joint
- removed joint FR_Knee_joint
- removed joint HL_HipX_joint
- removed joint HL_HipY_joint
- removed joint HL_Knee_joint
- removed joint HR_HipX_joint
- removed joint HR_HipY_joint
- removed joint HR_Knee_joint
- added joint FL_HipX: type revolute, parent TORSO, child FL_HIP, origin xyz=0.291 0.08 0 rpy=0 0 0, axis -1 0 0, limit lower=-0.323 upper=0.323 effort=84 velocity=17.5
- added joint FL_HipY: type revolute, parent FL_HIP, child FL_THIGH, origin xyz=0 0.11675 0 rpy=0 0 0, axis 0 -1 0, limit lower=-2.967 upper=0.262 effort=84 velocity=17.5
- added joint FL_Knee: type revolute, parent FL_THIGH, child FL_SHANK, origin xyz=0 0 -0.30 rpy=0 0 0, axis 0 -1 0, limit lower=0.349 upper=2.531 effort=160 velocity=16.1
- added joint FR_HipX: type revolute, parent TORSO, child FR_HIP, origin xyz=0.291 -0.08 0 rpy=0 0 0, axis -1 0 0, limit lower=-0.323 upper=0.323 effort=84 velocity=17.5
- added joint FR_HipY: type revolute, parent FR_HIP, child FR_THIGH, origin xyz=0 -0.11675 0 rpy=0 0 0, axis 0 -1 0, limit lower=-2.967 upper=0.262 effort=84 velocity=17.5
- added joint FR_Knee: type revolute, parent FR_THIGH, child FR_SHANK, origin xyz=0 0 -0.30 rpy=0 0 0, axis 0 -1 0, limit lower=0.349 upper=2.531 effort=160 velocity=16.1
- added joint HL_HipX: type revolute, parent TORSO, child HL_HIP, origin xyz=-0.291 0.08 0 rpy=0 0 0, axis -1 0 0, limit lower=-0.323 upper=0.323 effort=84 velocity=17.5
- added joint HL_HipY: type revolute, parent HL_HIP, child HL_THIGH, origin xyz=0 0.11675 0 rpy=0 0 0, axis 0 -1 0, limit lower=-2.967 upper=0.262 effort=84 velocity=17.5
- added joint HL_Knee: type revolute, parent HL_THIGH, child HL_SHANK, origin xyz=0 0 -0.30 rpy=0 0 0, axis 0 -1 0, limit lower=0.349 upper=2.531 effort=160 velocity=16.1
- added joint HR_HipX: type revolute, parent TORSO, child HR_HIP, origin xyz=-0.291 -0.08 0 rpy=0 0 0, axis -1 0 0, limit lower=-0.323 upper=0.323 effort=84 velocity=17.5
- added joint HR_HipY: type revolute, parent HR_HIP, child HR_THIGH, origin xyz=0 -0.11675 0 rpy=0 0 0, axis 0 -1 0, limit lower=-2.967 upper=0.262 effort=84 velocity=17.5
- added joint HR_Knee: type revolute, parent HR_THIGH, child HR_SHANK, origin xyz=0 0 -0.30 rpy=0 0 0, axis 0 -1 0, limit lower=0.349 upper=2.531 effort=160 velocity=16.1
- added joint floating_base: type fixed, parent base, child TORSO, origin xyz=0 0 0 rpy=0 0 0
- added joint imu_joint: type fixed, parent TORSO, child imu_link, origin xyz=0 0 0 rpy=0 0 0

File: descriptions/deep_robotics/x30_description/xacro/body.xacro (robot description, xacro)
@@ -52,5 +52,5 @@
     <child link="FL_HIP"/>
     <axis xyz="-1 0 0"/>
-    <limit lower="-0.323" upper="0.585" effort="84" velocity="17.5"/>
+    <limit lower="-0.323" upper="0.323" effort="84" velocity="17.5"/>
   </joint>
   <link name="FL_THIGH">
@@ -116,5 +116,5 @@
     <child link="FL_SHANK" />
     <axis xyz="0 -1 0" />
-    <limit lower="0.349" upper="2.531" effort="180" velocity="16.1" />
+    <limit lower="0.349" upper="2.531" effort="160" velocity="16.1" />
   </joint>
   <link name="FL_FOOT">
@@ -152,5 +152,5 @@
     <child link="FR_HIP" />
     <axis xyz="-1 0 0" />
-    <limit lower="-0.585" upper="0.323" effort="84" velocity="17.5" />
+    <limit lower="-0.323" upper="0.323" effort="84" velocity="17.5" />
   </joint>
   <link name="FR_THIGH">
@@ -216,5 +216,5 @@
     <child link="FR_SHANK" />
     <axis xyz="0 -1 0" />
-    <limit lower="0.349" upper="2.531" effort="180" velocity="16.1" />
+    <limit lower="0.349" upper="2.531" effort="160" velocity="16.1" />
   </joint>
   <link name="FR_FOOT">
@@ -252,5 +252,5 @@
     <child link="HL_HIP" />
     <axis xyz="-1 0 0" />
-    <limit lower="-0.323" upper="0.585" effort="84" velocity="17.5" />
+    <limit lower="-0.323" upper="0.323" effort="84" velocity="17.5" />
   </joint>
   <link name="HL_THIGH">
@@ -316,5 +316,5 @@
     <child link="HL_SHANK" />
     <axis xyz="0 -1 0" />
-    <limit lower="0.349" upper="2.531" effort="180" velocity="16.1" />
+    <limit lower="0.349" upper="2.531" effort="160" velocity="16.1" />
   </joint>
   <link name="HL_FOOT">
@@ -352,5 +352,5 @@
     <child link="HR_HIP" />
     <axis xyz="-1 0 0" />
-    <limit lower="-0.585" upper="0.323" effort="84" velocity="17.5" />
+    <limit lower="-0.323" upper="0.323" effort="84" velocity="17.5" />
   </joint>
   <link name="HR_THIGH">
@@ -416,5 +416,5 @@
     <child link="HR_SHANK" />
     <axis xyz="0 -1 0" />
-    <limit lower="0.349" upper="2.531" effort="180" velocity="16.1" />
+    <limit lower="0.349" upper="2.531" effort="160" velocity="16.1" />
   </joint>
   <link name="HR_FOOT">

Commit message: add relative path for ocs2 shared library

File: descriptions/deep_robotics/x30_description/urdf/robot.urdf (robot description, URDF)
Before this commit: robot x30, 19 links, 18 joints
Links:
- link TORSO: mass 30.7 -> 33.868

File: descriptions/unitree/go2_description/xacro/gazebo.xacro (robot description, xacro)
@@ -162,5 +162,5 @@
     <sensor name="imu_sensor" type="imu">
       <always_on>1</always_on>
-      <update_rate>500</update_rate>
+      <update_rate>1000</update_rate>
       <visualize>true</visualize>
       <topic>imu</topic>
