Commit message: migrate gz quadruped plugin to humble

File: descriptions/unitree/go2_description/urdf/robot.urdf (robot description, URDF)
Before this commit: robot go2, 19 links, 18 joints
Links:
- link FL_calf: geometry collision box size=0.213 0.016 0.016; visual mesh filename=../meshes/calf.dae scale=1 1 1
- link FL_hip: geometry collision cylinder length=0.04 radius=0.046; visual mesh filename=../meshes/hip.dae scale=1 1 1
- link FL_thigh: geometry collision box size=0.213 0.0245 0.034; visual mesh filename=../meshes/thigh.dae scale=1 1 1
- link FR_calf: geometry collision box size=0.213 0.016 0.016; visual mesh filename=../meshes/calf.dae scale=1 1 1
- link FR_hip: geometry collision cylinder length=0.04 radius=0.046; visual mesh filename=../meshes/hip.dae scale=1 1 1
- link FR_thigh: geometry collision box size=0.213 0.0245 0.034; visual mesh filename=../meshes/thigh_mirror.dae scale=1 1 1
- link RL_calf: geometry collision box size=0.213 0.016 0.016; visual mesh filename=../meshes/calf.dae scale=1 1 1
- link RL_hip: geometry collision cylinder length=0.04 radius=0.046; visual mesh filename=../meshes/hip.dae scale=1 1 1
- link RL_thigh: geometry collision box size=0.213 0.0245 0.034; visual mesh filename=../meshes/thigh.dae scale=1 1 1
- link RR_calf: geometry collision box size=0.213 0.016 0.016; visual mesh filename=../meshes/calf.dae scale=1 1 1
- link RR_hip: geometry collision cylinder length=0.04 radius=0.046; visual mesh filename=../meshes/hip.dae scale=1 1 1
- link RR_thigh: geometry collision box size=0.213 0.0245 0.034; visual mesh filename=../meshes/thigh_mirror.dae scale=1 1 1
- link trunk: geometry collision box size=0.3762 0.0935 0.114; visual mesh filename=../meshes/trunk.dae scale=1 1 1

Commit message: able to run gazebo simulation for ocs2 under humble

File: descriptions/unitree/go2_description/urdf/robot.urdf (robot description, URDF)
Before this commit: robot go2, 19 links, 18 joints
Links:
- link imu_link: geometry collision box size=0.001 0.001 0.001; visual box size=0.001 0.001 0.001
Joints:
- joint FL_calf_joint: origin xyz=0 0 -0.213 rpy=0 0 0 -> xyz=0 0 -0.213 rpy=0 -0 0
- joint FL_foot_fixed: axis (none) -> 0 0 0; origin xyz=0 0 -0.213 rpy=0 0 0 -> xyz=0 0 -0.213 rpy=0 -0 0
- joint FL_hip_joint: origin xyz=0.1934 0.0465 0 rpy=0 0 0 -> xyz=0.1934 0.0465 0 rpy=0 -0 0
- joint FL_thigh_joint: origin xyz=0 0.0955 0 rpy=0 0 0 -> xyz=0 0.0955 0 rpy=0 -0 0
- joint FR_calf_joint: origin xyz=0 0 -0.213 rpy=0 0 0 -> xyz=0 0 -0.213 rpy=0 -0 0
- joint FR_foot_fixed: axis (none) -> 0 0 0; origin xyz=0 0 -0.213 rpy=0 0 0 -> xyz=0 0 -0.213 rpy=0 -0 0
- joint FR_hip_joint: origin xyz=0.1934 -0.0465 0 rpy=0 0 0 -> xyz=0.1934 -0.0465 0 rpy=0 -0 0
- joint FR_thigh_joint: origin xyz=0 -0.0955 0 rpy=0 0 0 -> xyz=0 -0.0955 0 rpy=0 -0 0
- joint RL_calf_joint: origin xyz=0 0 -0.213 rpy=0 0 0 -> xyz=0 0 -0.213 rpy=0 -0 0
- joint RL_foot_fixed: axis (none) -> 0 0 0; origin xyz=0 0 -0.213 rpy=0 0 0 -> xyz=0 0 -0.213 rpy=0 -0 0
- joint RL_hip_joint: origin xyz=-0.1934 0.0465 0 rpy=0 0 0 -> xyz=-0.1934 0.0465 0 rpy=0 -0 0
- joint RL_thigh_joint: origin xyz=0 0.0955 0 rpy=0 0 0 -> xyz=0 0.0955 0 rpy=0 -0 0
- joint RR_calf_joint: origin xyz=0 0 -0.213 rpy=0 0 0 -> xyz=0 0 -0.213 rpy=0 -0 0
- joint RR_foot_fixed: axis (none) -> 0 0 0; origin xyz=0 0 -0.213 rpy=0 0 0 -> xyz=0 0 -0.213 rpy=0 -0 0
- joint RR_hip_joint: origin xyz=-0.1934 -0.0465 0 rpy=0 0 0 -> xyz=-0.1934 -0.0465 0 rpy=0 -0 0
- joint RR_thigh_joint: origin xyz=0 -0.0955 0 rpy=0 0 0 -> xyz=0 -0.0955 0 rpy=0 -0 0
- joint floating_base: axis (none) -> 0 0 0; origin xyz=0 0 0 rpy=0 0 0 -> xyz=0 0 0 rpy=0 -0 0
- joint imu_joint: axis (none) -> 0 0 0; origin xyz=0 0 0 rpy=0 0 0 -> xyz=0 0 0 rpy=0 -0 0
