Commit message: rename unitree sdk2 hardware, add gazebo for cyberdog

File: descriptions/anybotics/anymal_c_description/xacro/ros2_control.xacro (robot description, xacro)
@@ -3,5 +3,5 @@
   <ros2_control name="UnitreeSystem" type="system">
     <hardware>
-      <plugin>hardware_unitree_mujoco/HardwareUnitree</plugin>
+      <plugin>hardware_unitree_sdk2/HardwareUnitree</plugin>
     </hardware>
     <joint name="RF_HAA">

File: descriptions/deep_robotics/lite3_description/xacro/ros2_control.xacro (robot description, xacro)
@@ -3,5 +3,5 @@
   <ros2_control name="UnitreeSystem" type="system">
     <hardware>
-      <plugin>hardware_unitree_mujoco/HardwareUnitree</plugin>
+      <plugin>hardware_unitree_sdk2/HardwareUnitree</plugin>
     </hardware>
     <joint name="FR_HipX">

File: descriptions/unitree/a1_description/xacro/ros2_control.xacro (robot description, xacro)
@@ -3,5 +3,5 @@
   <ros2_control name="UnitreeSystem" type="system">
     <hardware>
-      <plugin>hardware_unitree_mujoco/HardwareUnitree</plugin>
+      <plugin>hardware_unitree_sdk2/HardwareUnitree</plugin>
     </hardware>
     <joint name="FR_hip_joint">

File: descriptions/unitree/b2_description/xacro/ros2_control.xacro (robot description, xacro)
@@ -3,5 +3,5 @@
     <ros2_control name="UnitreeSystem" type="system">
         <hardware>
-            <plugin>hardware_unitree_mujoco/HardwareUnitree</plugin>
+            <plugin>hardware_unitree_sdk2/HardwareUnitree</plugin>
         </hardware>
         <joint name="FR_hip_joint">

File: descriptions/unitree/go1_description/xacro/ros2_control.xacro (robot description, xacro)
@@ -3,5 +3,5 @@
 	<ros2_control name="UnitreeSystem" type="system">
 		<hardware>
-			<plugin>hardware_unitree_mujoco/HardwareUnitree</plugin>
+			<plugin>hardware_unitree_sdk2/HardwareUnitree</plugin>
 		</hardware>
 		<joint name="FR_hip_joint">

File: descriptions/unitree/go2_description/xacro/gazebo.xacro (robot description, xacro)
@@ -149,7 +149,5 @@
       <parameters>$(find go2_description)/config/gazebo.yaml</parameters>
     </plugin>
-    <plugin filename="gz-sim-imu-system"
-            name="gz::sim::systems::Imu">
-    </plugin>
+    <plugin filename="gz-sim-imu-system" name="gz::sim::systems::Imu"/>
     <plugin filename="gz-sim-forcetorque-system" name="gz::sim::systems::ForceTorque"/>
   </gazebo>

File: descriptions/unitree/go2_description/xacro/ros2_control.xacro (robot description, xacro)
@@ -3,5 +3,5 @@
 	<ros2_control name="UnitreeSystem" type="system">
 		<hardware>
-			<plugin>hardware_unitree_mujoco/HardwareUnitree</plugin>
+			<plugin>hardware_unitree_sdk2/HardwareUnitree</plugin>
 <!--			<param name="domain">0</param>-->
 <!--			<param name="network_interface">enp46s0</param>-->

File: descriptions/xiaomi/cyberdog_description/xacro/const.xacro (robot description, xacro)
@@ -47,7 +47,7 @@
   <xacro:property name="hip_motorVelMax" value="30.9971"/>
   <xacro:property name="knee_motorVelMax" value="30.9971"/>
-  <xacro:property name="abad_damping" value="0.1"/>
-  <xacro:property name="hip_damping" value="0.1"/>
-  <xacro:property name="knee_damping" value="0.1"/>
+  <xacro:property name="abad_damping" value="0.01"/>
+  <xacro:property name="hip_damping" value="0.01"/>
+  <xacro:property name="knee_damping" value="0.01"/>
   <xacro:property name="abad_friction" value="0.1"/>
   <xacro:property name="hip_friction" value="0.1"/>
@@ -109,3 +109,4 @@
   <xacro:property name="rotor_iyz" value="0"/>
   <xacro:property name="rotor_izz" value="0.000025300"/>
+  <xacro:property name="foot_mass" value="0.06"/>
 </robot>

File: descriptions/xiaomi/cyberdog_description/xacro/gazebo.xacro (robot description, xacro)
@@ -3,8 +3,12 @@
   <ros2_control name="GazeboSystem" type="system">
     <hardware>
-      <plugin>gz_ros2_control/GazeboSimSystem</plugin>
+      <plugin>gz_quadruped_hardware/GazeboSimSystem</plugin>
     </hardware>
     <joint name="FR_hip_joint">
-      <command_interface name="effort" initial_value="0.0"/>
+      <command_interface name="position"/>
+      <command_interface name="velocity"/>
+      <command_interface name="effort"/>
+      <command_interface name="kp"/>
+      <command_interface name="kd"/>
       <state_interface name="position"/>
       <state_interface name="velocity"/>
@@ -12,5 +16,9 @@
     </joint>
     <joint name="FR_thigh_joint">
-      <command_interface name="effort" initial_value="0.0"/>
+      <command_interface name="position"/>
+      <command_interface name="velocity"/>
+      <command_interface name="effort"/>
+      <command_interface name="kp"/>
+      <command_interface name="kd"/>
       <state_interface name="position"/>
       <state_interface name="velocity"/>
@@ -18,5 +26,9 @@
     </joint>
     <joint name="FR_calf_joint">
-      <command_interface name="effort" initial_value="0.0"/>
+      <command_interface name="position"/>
+      <command_interface name="velocity"/>
+      <command_interface name="effort"/>
+      <command_interface name="kp"/>
+      <command_interface name="kd"/>
       <state_interface name="position"/>
       <state_interface name="velocity"/>
@@ -24,5 +36,9 @@
     </joint>
     <joint name="FL_hip_joint">
-      <command_interface name="effort" initial_value="0.0"/>
+      <command_interface name="position"/>
+      <command_interface name="velocity"/>
+      <command_interface name="effort"/>
+      <command_interface name="kp"/>
+      <command_interface name="kd"/>
       <state_interface name="position"/>
       <state_interface name="velocity"/>
@@ -30,5 +46,9 @@
     </joint>
     <joint name="FL_thigh_joint">
-      <command_interface name="effort" initial_value="0.0"/>
+      <command_interface name="position"/>
+      <command_interface name="velocity"/>
+      <command_interface name="effort"/>
+      <command_interface name="kp"/>
+      <command_interface name="kd"/>
       <state_interface name="position"/>
       <state_interface name="velocity"/>
@@ -36,5 +56,9 @@
     </joint>
     <joint name="FL_calf_joint">
-      <command_interface name="effort" initial_value="0.0"/>
+      <command_interface name="position"/>
+      <command_interface name="velocity"/>
+      <command_interface name="effort"/>
+      <command_interface name="kp"/>
+      <command_interface name="kd"/>
       <state_interface name="position"/>
       <state_interface name="velocity"/>
@@ -42,5 +66,9 @@
     </joint>
     <joint name="RR_hip_joint">
-      <command_interface name="effort" initial_value="0.0"/>
+      <command_interface name="position"/>
+      <command_interface name="velocity"/>
+      <command_interface name="effort"/>
+      <command_interface name="kp"/>
+      <command_interface name="kd"/>
       <state_interface name="position"/>
       <state_interface name="velocity"/>
@@ -48,5 +76,9 @@
     </joint>
     <joint name="RR_thigh_joint">
-      <command_interface name="effort" initial_value="0.0"/>
+      <command_interface name="position"/>
+      <command_interface name="velocity"/>
+      <command_interface name="effort"/>
+      <command_interface name="kp"/>
+      <command_interface name="kd"/>
       <state_interface name="position"/>
       <state_interface name="velocity"/>
@@ -54,5 +86,9 @@
     </joint>
     <joint name="RR_calf_joint">
-      <command_interface name="effort" initial_value="0.0"/>
+      <command_interface name="position"/>
+      <command_interface name="velocity"/>
+      <command_interface name="effort"/>
+      <command_interface name="kp"/>
+      <command_interface name="kd"/>
       <state_interface name="position"/>
       <state_interface name="velocity"/>
@@ -60,5 +96,9 @@
     </joint>
     <joint name="RL_hip_joint">
-      <command_interface name="effort" initial_value="0.0"/>
+      <command_interface name="position"/>
+      <command_interface name="velocity"/>
+      <command_interface name="effort"/>
+      <command_interface name="kp"/>
+      <command_interface name="kd"/>
       <state_interface name="position"/>
       <state_interface name="velocity"/>
@@ -66,5 +106,9 @@
     </joint>
     <joint name="RL_thigh_joint">
-      <command_interface name="effort" initial_value="0.0"/>
+      <command_interface name="position"/>
+      <command_interface name="velocity"/>
+      <command_interface name="effort"/>
+      <command_interface name="kp"/>
+      <command_interface name="kd"/>
       <state_interface name="position"/>
       <state_interface name="velocity"/>
@@ -72,5 +116,9 @@
     </joint>
     <joint name="RL_calf_joint">
-      <command_interface name="effort" initial_value="0.0"/>
+      <command_interface name="position"/>
+      <command_interface name="velocity"/>
+      <command_interface name="effort"/>
+      <command_interface name="kp"/>
+      <command_interface name="kd"/>
       <state_interface name="position"/>
       <state_interface name="velocity"/>
@@ -89,43 +137,18 @@
       <state_interface name="linear_acceleration.z"/>
     </sensor>
-    <sensor name="LF_foot_end">
-      <state_interface name="force.x"/>
-      <state_interface name="force.y"/>
-      <state_interface name="force.z"/>
-      <param name="frame_id">LF_FOOT</param>
-    </sensor>
-    <sensor name="RF_foot_end">
-      <state_interface name="force.x"/>
-      <state_interface name="force.y"/>
-      <state_interface name="force.z"/>
-      <param name="frame_id">RF_FOOT</param>
-    </sensor>
-    <sensor name="LH_foot_end">
-      <state_interface name="force.x"/>
-      <state_interface name="force.y"/>
-      <state_interface name="force.z"/>
-      <param name="frame_id">LH_FOOT</param>
-    </sensor>
-    <sensor name="RH_foot_end">
-      <state_interface name="force.x"/>
-      <state_interface name="force.y"/>
-      <state_interface name="force.z"/>
-      <param name="frame_id">LH_FOOT</param>
+    <sensor name="foot_force">
+      <state_interface name="FR_foot_force"/>
+      <state_interface name="FL_foot_force"/>
+      <state_interface name="RR_foot_force"/>
+      <state_interface name="RL_foot_force"/>
     </sensor>
   </ros2_control>
   <!-- Gazebo's ros2_control plugin  -->
   <gazebo>
-    <plugin filename="gz_ros2_control-system" name="gz_ros2_control::GazeboSimROS2ControlPlugin">
+    <plugin filename="gz_quadruped_hardware-system" name="gz_quadruped_hardware::GazeboSimQuadrupedPlugin">
       <parameters>$(find cyberdog_description)/config/gazebo.yaml</parameters>
     </plugin>
-    <plugin filename="gz-sim-imu-system"
-            name="gz::sim::systems::Imu">
-    </plugin>
-    <plugin filename="gz-sim-contact-system"
-            name="gz::sim::systems::Contact">
-    </plugin>
-    <plugin filename="gz-sim-forcetorque-system"
-            name="gz::sim::systems::ForceTorque">
-    </plugin>
+    <plugin filename="gz-sim-imu-system" name="gz::sim::systems::Imu"/>
+    <plugin filename="gz-sim-forcetorque-system" name="gz::sim::systems::ForceTorque"/>
   </gazebo>
   <gazebo reference="imu_link">
@@ -194,3 +217,8 @@
     <disableFixedJointLumping>true</disableFixedJointLumping>
   </gazebo>
+  <xacro:include filename="$(find gz_quadruped_hardware)/xacro/foot_force_sensor.xacro"/>
+  <xacro:foot_force_sensor name="FL" suffix="foot_fixed"/>
+  <xacro:foot_force_sensor name="RL" suffix="foot_fixed"/>
+  <xacro:foot_force_sensor name="FR" suffix="foot_fixed"/>
+  <xacro:foot_force_sensor name="RR" suffix="foot_fixed"/>
 </robot>

File: descriptions/xiaomi/cyberdog_description/xacro/leg.xacro (robot description, xacro)
@@ -213,13 +213,12 @@
           <sphere radius="${foot_radius}"/>
         </geometry>
-        <surface>
-          <contact>
-            <ode>
-              <max_vel>0.001</max_vel>
-              <min_depth>0.0</min_depth>
-            </ode>
-          </contact>
-        </surface>
-      </collision>
+      </collision>
+      <inertial>
+        <mass value="${foot_mass}"/>
+        <inertia
+            ixx="${(2*foot_mass)/5.0*(foot_radius*foot_radius)}" ixy="0.0" ixz="0.0"
+            iyy="${(2*foot_mass)/5.0*(foot_radius*foot_radius)}" iyz="0.0"
+            izz="${(2*foot_mass)/5.0*(foot_radius*foot_radius)}"/>
+      </inertial>
     </link>
     <xacro:leg_transmission name="${name}"/>
@@ -227,11 +226,4 @@
       <mu1>0.2</mu1>
       <mu2>0.2</mu2>
-      <visual>
-        <material>
-          <ambient>.5 .5 .5 1.0</ambient>
-          <diffuse>.5 .5 .5 1.0</diffuse>
-          <specular>.5 .5 .5 1.0</specular>
-        </material>
-      </visual>
     </gazebo>
     <gazebo reference="${name}_hip">
@@ -239,11 +231,6 @@
       <mu2>0.2</mu2>
       <self_collide>1</self_collide>
-      <visual>
-        <material>
-          <ambient>.05 .05 .05 1.0</ambient>
-          <diffuse>.05 .05 .05 1.0</diffuse>
-          <specular>.05 .05 .05 1.0</specular>
-        </material>
-      </visual>
+      <kp value="1000000.0"/>
+      <kd value="100.0"/>
     </gazebo>
     <gazebo reference="${name}_knee">
@@ -251,11 +238,4 @@
       <mu2>0.7</mu2>
       <self_collide>1</self_collide>
-      <visual>
-        <material>
-          <ambient>.5 .5 .5 1.0</ambient>
-          <diffuse>.5 .5 .5 1.0</diffuse>
-          <specular>.5 .5 .5 1.0</specular>
-        </material>
-      </visual>
     </gazebo>
     <gazebo reference="${name}_foot">
@@ -263,11 +243,6 @@
       <mu2>0.7</mu2>
       <self_collide>1</self_collide>
-      <visual>
-        <material>
-          <ambient>.5 .5 .5 1.0</ambient>
-          <diffuse>.5 .5 .5 1.0</diffuse>
-          <specular>.5 .5 .5 1.0</specular>
-        </material>
-      </visual>
+      <kp value="1000000.0"/>
+      <kd value="100.0"/>
     </gazebo>
   </xacro:macro>
